File: esempi/04_motor_driver_LD293D/04_motor_driver_L293D.sch (KiCad schematic (older format))
At the start: 13 parts, among them IC1 L293D, P1 MOTOR1_DIRECTION, P2 MOTOR1_ENABLE, P3 CONN_01X02, P4 MOTOR2_ENABLE, P5 CONN_01X02, P6 MOTOR2_DIRECTION, Q1 Q_NPN_BCE, Q2 Q_NPN_BCE

Commit message: Aggiunti esempi nuovo componente, arduino shield, modoficato motor driver
Parts:
- added P7, P8, P9: CONN_01X01, w_pin_strip:pin_strip_1, symbol CONN_01X01
- P1, P2, P4, P6: footprint Pin_Headers:Pin_Header_Straight_1x01 -> w_pin_strip:pin_strip_1
- P3, P5: footprint Pin_Headers:Pin_Header_Straight_1x02 -> w_pin_strip:pin_strip_2
- R1, R2, R3, R4: footprint w_pth_resistors:R15.5x6_vert -> w_pth_resistors:R12x5.2
Connections:
- net +5V: now also P8.1 (P1)
- net GND: now also P9.1 (P1)
- net VCC: now also P7.1 (P1)
Changed lines of the file:
@@
 LIBS:valves
 LIBS:stepper drivers
+LIBS:04_motor_driver_L293D-cache
 EELAYER 25 0
 EELAYER END
@@
 F 0 "P3" H 3150 3200 50  0000 C CNN
 F 1 "CONN_01X02" V 3250 3050 50  0000 C CNN
-F 2 "Pin_Headers:Pin_Header_Straight_1x02" H 3150 3050 60  0001 C CNN
+F 2 "w_pin_strip:pin_strip_2" H 3150 3050 60  0001 C CNN
 F 3 "" H 3150 3050 60  0000 C CNN
 	1    3150 3050
@@
 F 0 "P4" H 5600 3850 50  0000 C CNN
 F 1 "MOTOR2_ENABLE" H 5600 3550 50  0000 C CNN
-F 2 "Pin_Headers:Pin_Header_Straight_1x01" H 5600 3750 60  0001 C CNN
+F 2 "w_pin_strip:pin_strip_1" H 5600 3750 60  0001 C CNN
 F 3 "" H 5600 3750 60  0000 C CNN
 	1    5600 3750
@@
 F 0 "P2" H 3150 2450 50  0000 C CNN
 F 1 "MOTOR1_ENABLE" H 3150 2200 50  0000 C CNN
-F 2 "Pin_Headers:Pin_Header_Straight_1x01" H 3150 2350 60  0001 C CNN
+F 2 "w_pin_strip:pin_strip_1" H 3150 2350 60  0001 C CNN
 F 3 "" H 3150 2350 60  0000 C CNN
 	1    3150 2350
@@
 F 0 "R2" V 2730 2850 50  0000 C CNN
 F 1 "R" V 2650 2850 50  0000 C CNN
-F 2 "w_pth_resistors:R15.5x6_vert" V 2580 2850 30  0001 C CNN
+F 2 "w_pth_resistors:R12x5.2" V 2580 2850 30  0001 C CNN
 F 3 "" H 2650 2850 30  0000 C CNN
 	1    2650 2850
@@
 F 0 "R1" V 2380 2850 50  0000 C CNN
 F 1 "R" V 2300 2850 50  0000 C CNN
-F 2 "w_pth_resistors:R15.5x6_vert" V 2230 2850 30  0001 C CNN
+F 2 "w_pth_resistors:R12x5.2" V 2230 2850 30  0001 C CNN
 F 3 "" H 2300 2850 30  0000 C CNN
 	1    2300 2850
@@
 F 0 "P1" H 1900 2650 50  0000 C CNN
 F 1 "MOTOR1_DIRECTION" H 1900 2400 50  0000 C CNN
-F 2 "Pin_Headers:Pin_Header_Straight_1x01" H 1900 2550 60  0001 C CNN
+F 2 "w_pin_strip:pin_strip_1" H 1900 2550 60  0001 C CNN
 F 3 "" H 1900 2550 60  0000 C CNN
 	1    1900 2550
@@
 F 0 "P5" H 6250 3200 50  0000 C CNN
 F 1 "CONN_01X02" V 6350 3050 50  0000 C CNN
-F 2 "Pin_Headers:Pin_Header_Straight_1x02" H 6250 3050 60  0001 C CNN
+F 2 "w_pin_strip:pin_strip_2" H 6250 3050 60  0001 C CNN
 F 3 "" H 6250 3050 60  0000 C CNN
 	1    6250 3050
@@
 F 0 "R3" V 6830 2850 50  0000 C CNN
 F 1 "R" V 6750 2850 50  0000 C CNN
-F 2 "w_pth_resistors:R15.5x6_vert" V 6680 2850 30  0001 C CNN
+F 2 "w_pth_resistors:R12x5.2" V 6680 2850 30  0001 C CNN
 F 3 "" H 6750 2850 30  0000 C CNN
 	1    6750 2850
@@
 F 0 "R4" V 7180 2850 50  0000 C CNN
 F 1 "R" V 7100 2850 50  0000 C CNN
-F 2 "w_pth_resistors:R15.5x6_vert" V 7030 2850 30  0001 C CNN
+F 2 "w_pth_resistors:R12x5.2" V 7030 2850 30  0001 C CNN
 F 3 "" H 7100 2850 30  0000 C CNN
 	1    7100 2850
@@
 F 0 "P6" H 7500 2650 50  0000 C CNN
 F 1 "MOTOR2_DIRECTION" H 7500 2400 50  0000 C CNN
-F 2 "Pin_Headers:Pin_Header_Straight_1x01" H 7500 2550 60  0001 C CNN
+F 2 "w_pin_strip:pin_strip_1" H 7500 2550 60  0001 C CNN
 F 3 "" H 7500 2550 60  0000 C CNN
 	1    7500 2550
@@
 	3650 3900 3650 4000
 Wire Wire Line
-	3650 4000 3850 4000
+	3600 4000 3850 4000
 Connection ~ 3850 4000
 Wire Wire Line
 	2650 4200 2650 4050
+$Comp
+L CONN_01X01 P8
+U 1 1 55410F7D
+P 4700 1700
+F 0 "P8" H 4700 1800 50  0000 C CNN
+F 1 "CONN_01X01" V 4800 1700 50  0000 C CNN
+F 2 "w_pin_strip:pin_strip_1" H 4700 1700 60  0001 C CNN
+F 3 "" H 4700 1700 60  0000 C CNN
+	1    4700 1700
+	0    -1   -1   0
+$EndComp
+Wire Wire Line
+	4700 1900 4700 2000
+Connection ~ 4700 2000
+$Comp
+L CONN_01X01 P7
+U 1 1 55411081
+P 3400 4000
+F 0 "P7" H 3400 4100 50  0000 C CNN
+F 1 "CONN_01X01" V 3500 4000 50  0000 C CNN
+F 2 "w_pin_strip:pin_strip_1" H 3400 4000 60  0001 C CNN
+F 3 "" H 3400 4000 60  0000 C CNN
+	1    3400 4000
+	-1   0    0    1
+$EndComp
+Connection ~ 3650 4000
+$Comp
+L CONN_01X01 P9
+U 1 1 554111FC
+P 6300 4350
+F 0 "P9" H 6300 4450 50  0000 C CNN
+F 1 "CONN_01X01" V 6400 4350 50  0000 C CNN
+F 2 "w_pin_strip:pin_strip_1" H 6300 4350 60  0001 C CNN
+F 3 "" H 6300 4350 60  0000 C CNN
+	1    6300 4350
+	0    1    1    0
+$EndComp
+Wire Wire Line
+	6300 4150 6750 4150
+Connection ~ 6750 4150
 $EndSCHEMATC
