File: esempi/04_motor_driver_LD293D/_saved_04_motor_driver_L293D.sch (KiCad schematic (older format))
At the start: 20 parts, among them IC1 L293D, P1 MOTOR1_DIRECTION, P2 MOTOR1_ENABLE, P3 CONN_01X02, P4 MOTOR2_ENABLE, P5 CONN_01X02, P6 MOTOR2_DIRECTION, P7 CONN_01X01, P8 CONN_01X01, P9 CONN_01X01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

Commit message: sistemato circuito L293D
Parts:
- R1, R2, R3, R4: footprint w_pth_resistors:R12x5.2 -> w_pth_resistors:RC03
Changed lines of the file:
@@
 F 0 "R2" V 2730 2850 50  0000 C CNN
 F 1 "R" V 2650 2850 50  0000 C CNN
-F 2 "w_pth_resistors:R12x5.2" V 2580 2850 30  0001 C CNN
+F 2 "w_pth_resistors:RC03" V 2580 2850 30  0001 C CNN
 F 3 "" H 2650 2850 30  0000 C CNN
 	1    2650 2850
@@
 F 0 "R1" V 2380 2850 50  0000 C CNN
 F 1 "R" V 2300 2850 50  0000 C CNN
-F 2 "w_pth_resistors:R12x5.2" V 2230 2850 30  0001 C CNN
+F 2 "w_pth_resistors:RC03" V 2230 2850 30  0001 C CNN
 F 3 "" H 2300 2850 30  0000 C CNN
 	1    2300 2850
@@
 F 0 "R3" V 6830 2850 50  0000 C CNN
 F 1 "R" V 6750 2850 50  0000 C CNN
-F 2 "w_pth_resistors:R12x5.2" V 6680 2850 30  0001 C CNN
+F 2 "w_pth_resistors:RC03" V 6680 2850 30  0001 C CNN
 F 3 "" H 6750 2850 30  0000 C CNN
 	1    6750 2850
@@
 F 0 "R4" V 7180 2850 50  0000 C CNN
 F 1 "R" V 7100 2850 50  0000 C CNN
-F 2 "w_pth_resistors:R12x5.2" V 7030 2850 30  0001 C CNN
+F 2 "w_pth_resistors:RC03" V 7030 2850 30  0001 C CNN
 F 3 "" H 7100 2850 30  0000 C CNN
 	1    7100 2850
