File: esempi/08_arduino_shield/08_arduino_shield.sch (KiCad schematic (older format))
At the start: 7 parts, among them J1 Arduino_Header, P1 CONN_01X02, U1 ULN2803

Commit message: Modifiche ad arduino shield per connettori più piccoli
Parts:
- L1, L2, L3, L4, P1: footprint w_conn_gmkds:gmkds_3-2-7,62 -> w_conn_screw:mors_2p
Changed lines of the file:
@@
 LIBS:w_transistor
 LIBS:w_vacuum
+LIBS:08_arduino_shield-cache
 EELAYER 25 0
 EELAYER END
@@
 F 0 "L1" H 7650 2850 50  0000 C CNN
 F 1 "INDUCTOR_SMALL" H 7650 2700 50  0000 C CNN
-F 2 "w_conn_gmkds:gmkds_3-2-7,62" H 7650 2750 60  0001 C CNN
+F 2 "w_conn_screw:mors_2p" H 7650 2750 60  0001 C CNN
 F 3 "" H 7650 2750 60  0000 C CNN
 	1    7650 2750
@@
 F 0 "L2" H 8050 2850 50  0000 C CNN
 F 1 "INDUCTOR_SMALL" H 8050 2700 50  0000 C CNN
-F 2 "w_conn_gmkds:gmkds_3-2-7,62" H 8050 2750 60  0001 C CNN
+F 2 "w_conn_screw:mors_2p" H 8050 2750 60  0001 C CNN
 F 3 "" H 8050 2750 60  0000 C CNN
 	1    8050 2750
@@
 F 0 "L3" H 8450 2850 50  0000 C CNN
 F 1 "INDUCTOR_SMALL" H 8450 2700 50  0000 C CNN
-F 2 "w_conn_gmkds:gmkds_3-2-7,62" H 8450 2750 60  0001 C CNN
+F 2 "w_conn_screw:mors_2p" H 8450 2750 60  0001 C CNN
 F 3 "" H 8450 2750 60  0000 C CNN
 	1    8450 2750
@@
 F 0 "L4" H 8850 2850 50  0000 C CNN
 F 1 "INDUCTOR_SMALL" H 8850 2700 50  0000 C CNN
-F 2 "w_conn_gmkds:gmkds_3-2-7,62" H 8850 2750 60  0001 C CNN
+F 2 "w_conn_screw:mors_2p" H 8850 2750 60  0001 C CNN
 F 3 "" H 8850 2750 60  0000 C CNN
 	1    8850 2750
@@
 F 0 "P1" H 9750 3750 50  0000 C CNN
 F 1 "CONN_01X02" V 9850 3600 50  0000 C CNN
-F 2 "w_conn_gmkds:gmkds_3-2-7,62" H 9750 3600 60  0001 C CNN
+F 2 "w_conn_screw:mors_2p" H 9750 3600 60  0001 C CNN
 F 3 "" H 9750 3600 60  0000 C CNN
 	1    9750 3600
